Commit message: Moodul 02: minu_description + sonar_link + vastused

File: minu_description/urdf/yahboom_robot.urdf.xacro (robot description, xacro)
@@ -212,3 +212,22 @@
     4. Miks on mõlemat vaja?
   -->
+<!-- SONAR -->
+<link name="sonar_link">
+  <visual>
+    <geometry>
+      <box size="0.05 0.05 0.05"/>
+    </geometry>
+  </visual>
+  <collision>
+    <geometry>
+      <box size="0.05 0.05 0.05"/>
+    </geometry>
+  </collision>
+  <xacro:box_inertia m="0.01" x="0.05" y="0.05" z="0.05"/>
+</link>
+<joint name="sonar_joint" type="fixed">
+  <parent link="base_link"/>
+  <child link="sonar_link"/>
+  <origin xyz="0.08 0 0.03" rpy="0 0 0"/>
+</joint>
 </robot>
